File: xiaomi-airpurifier-custom-board/xiaomi-airpurifier-custom-board.kicad_pcb (KiCad board)
At the start: 2 copper layers, 130 x 49 mm, 64 parts, among them J1 XY-VH3.96-2A21, J10 Conn_LD2410, J11 Conn_01x06_Pin, J2 JST S06B-PASK-2(LF)(SN), J3 B02B-PASK-1(LF)(SN), J4 BX-PH2.0-2PZZ, J5 HDGC2001WV-4P, J6 B07B-PASK(LF)(SN), J7 B04B-PASK-1(LF)(SN), J8 B05B-PASK-1(LF)(SN)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

Commit message: Add CI
Parts:
- removed JP1, JP2, JP3: SolderJumper_2_Bridged, Jumper:SolderJumper-2_P1.3mm_Bridged_RoundedPad1.0x1.5mm
- added J9: ~, Connector_JST:JST_PH_B4B-PH-K_1x04_P2.00mm_Vertical, F.Cu at (125.0, 15.0)
- added Q3: SS8050G, Package_TO_SOT_SMD:SOT-23, F.Cu at (29.0, 50.8)
- added R23: 10k, Resistor_SMD:R_0603_1608Metric, F.Cu at (25.2, 19.5)
- added R24: 20k, Resistor_SMD:R_0603_1608Metric, F.Cu at (25.2, 21.5)
- added R25: 10k, Resistor_SMD:R_0603_1608Metric, F.Cu at (28.8, 21.5)
- added R26: 20k, Resistor_SMD:R_0603_1608Metric, F.Cu at (28.8, 19.5)
- added R27: 1k, Resistor_SMD:R_0603_1608Metric, F.Cu at (33.0, 49.8)
- added R28: 10k, Resistor_SMD:R_0603_1608Metric, F.Cu at (26.0, 49.8)
- added TP1: TestPoint, TestPoint:TestPoint_Pad_D1.0mm, F.Cu at (132.0, 50.8)
- added TP2: TestPoint, TestPoint:TestPoint_Pad_D1.0mm, F.Cu at (135.5, 50.8)
- added TP3: TestPoint, TestPoint:TestPoint_Pad_D1.0mm, F.Cu at (120.8, 49.8)
- added TP4: TestPoint, TestPoint:TestPoint_Pad_D1.0mm, F.Cu at (125.5, 58.0)
- added TP5: TestPoint, TestPoint:TestPoint_Pad_D1.0mm, F.Cu at (127.5, 60.0)
- added kibuzzard-69EA09FB: G***, kibuzzard-69EA09FB, F.Cu at (16.8, 22.2)
- added kibuzzard-69EA0A86: G***, kibuzzard-69EA0A86, F.Cu at (31.2, 29.2)
- added kibuzzard-69EA0AD8: G***, kibuzzard-69EA0AD8, F.Cu at (31.2, 25.0)
- JP4, JP5: moved to B.Cu
- R1, R2: value 4.7k -> 5.1k 1%; footprint Resistor_SMD:R_0603_1608Metric_Pad0.98x0.95mm_HandSolder -> Resistor_SMD:R_0603_1608Metric
- moved JP4 70.0 mm to (27.0, 41.8), turned to 90 degrees
- moved JP5 63.4 mm to (29.8, 41.8), turned to 90 degrees
- moved R21 6.40 mm to (22.5, 50.0), turned to -90 degrees
- moved Q2 4.00 mm to (29.0, 54.5)
- moved R19 3.69 mm to (32.8, 57.2)
- moved R20 2.00 mm to (33.0, 53.5)
- moved R18 1.77 mm to (23.2, 41.2)
- moved R17 1.27 mm to (23.2, 45.0)
- moved R22 1.27 mm to (24.2, 49.8)
- moved Q1 1.03 mm to (29.0, 58.2), turned to 180 degrees
- moved C2 0.90 mm to (48.5, 28.8), turned to 90 degrees
- moved F1 0.50 mm to (23.8, 33.5)
Connections:
- C10 pad 1: Net-(JP5-A) -> +5V
- C9 pad 1: /3.3V_PRE_JUMPER -> +3.3V
- J8 pad 2: unconnected-(J8-Pin_2-Pad2) -> Net-(J8-Pin_2)
- J8 pad 4: /PM2_TX -> /PM2_PWM
- J8 pad 5: unconnected-(J8-Pin_5-Pad5) -> Net-(J8-Pin_5)
- JP4 pad 1: /3.3V_PRE_JUMPER -> Net-(J8-Pin_5)
- JP4 pad 2: +3.3V -> /PM2_RX
- JP5 pad 1: Net-(JP5-A) -> Net-(J8-Pin_2)
- JP5 pad 2: +5V -> /PM2_TX
- L1 pad 2: /3.3V_PRE_JUMPER -> +3.3V
- L2 pad 2: Net-(JP5-A) -> +5V
- R6 pad 2: /3.3V_PRE_JUMPER -> +3.3V
- R7 pad 2: Net-(JP5-A) -> +5V
- U3 pad 18: Net-(JP3-B) -> GND
- U3 pad 23: Net-(JP2-B) -> GND
- U3 pad 24: Net-(JP1-B) -> GND
- U4 pad 10: /PM2_TX -> /PM2_PWM_3.3V
- U4 pad 20: unconnected-(U4-GPIO15-Pad20) -> /PM2_RX_3.3V
- U4 pad 22: unconnected-(U4-GPIO8-Pad22) -> /IO8_EXTRA
- U4 pad 5: unconnected-(U4-GPIO2/ADC1_CH2-Pad5) -> /IO2_EXTRA
- U4 pad 6: unconnected-(U4-GPIO3/ADC1_CH3-Pad6) -> /PM2_TX_3.3V
- U5 pad A4: unconnected-(U5-VBUS-PadA4) -> /VBUS
- U5 pad A9: unconnected-(U5-VBUS-PadA9) -> /VBUS
- U5 pad B4: unconnected-(U5-VBUS-PadB4) -> /VBUS
- U5 pad B9: unconnected-(U5-VBUS-PadB9) -> /VBUS
Routing:
- net /PM2_PWM_3.3V: track 0.00 -> 124.7 mm, vias 0 -> 2
- net /PM2_TX_3.3V: track 0.00 -> 122.5 mm, vias 0 -> 2
- net /PM2_RX_3.3V: track 0.00 -> 105.2 mm, vias 0 -> 4
- net /PM2_TX: track 114.0 -> 25.8 mm
- net +5V: track 143.1 -> 174.6 mm
- net /PM2_PWM: track 0.00 -> 30.3 mm, vias 0 -> 1
- net /IO8_EXTRA: track 0.00 -> 28.9 mm, vias 0 -> 1
- net /VBUS: track 0.00 -> 19.1 mm
- net Net-(JP5-A): track 18.7 -> 0.00 mm
- net /3.3V_PRE_JUMPER: track 18.7 -> 0.00 mm
- net /IO2_EXTRA: track 0.00 -> 16.7 mm, vias 0 -> 1
- net /PM2_RX: track 0.00 -> 13.7 mm, vias 0 -> 1
- net +3.3V: track 198.7 -> 212.4 mm, vias 5 -> 3
- net /USB+: track 22.6 -> 30.1 mm
- net Net-(JP1-B): track 7.32 -> 0.00 mm
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Other:
- board text added: "${CI_BOARD_REPO_LINK}"
- board text added: "${CI_BOARD_REVISION}"
- board text added: "Air purifier board rev2 04.2026 alufers"
- board text added: "PM2_PWM"
- board text added: "PM2_RX"
- board text removed: "+"
- board text removed: "-"
- board text removed: "Air purifier board rev1 03.2026 alufers"
