File: xiaomi-airpurifier-custom-board/xiaomi-airpurifier-custom-board.kicad_sch (KiCad schematic)
At the start: 64 parts, among them J1 XY-VH3.96-2A21, J10 Conn_LD2410, J11 Conn_01x06_Pin, J2 JST S06B-PASK-2(LF)(SN), J3 B02B-PASK-1(LF)(SN), J4 BX-PH2.0-2PZZ, J5 HDGC2001WV-4P, J6 B07B-PASK(LF)(SN), J7 B04B-PASK-1(LF)(SN), J8 B05B-PASK-1(LF)(SN)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

Commit message: Add CI
Parts:
- removed JP1, JP2, JP3: SolderJumper_2_Bridged, Jumper:SolderJumper-2_P1.3mm_Bridged_RoundedPad1.0x1.5mm, symbol Jumper:SolderJumper_2_Bridged
- added J9: (no value), Connector_JST:JST_PH_B4B-PH-K_1x04_P2.00mm_Vertical, symbol Connector:Conn_01x04_Pin
- added Q3: SS8050G, Package_TO_SOT_SMD:SOT-23, symbol Transistor_BJT:SS8050
- added R23, R25, R28: 10k, Resistor_SMD:R_0603_1608Metric, symbol Device:R
- added R24, R26: 20k, Resistor_SMD:R_0603_1608Metric, symbol Device:R
- added R27: 1k, Resistor_SMD:R_0603_1608Metric, symbol Device:R
- added TP1, TP2, TP3, TP4, TP5: TestPoint, TestPoint:TestPoint_Pad_D1.0mm, symbol Connector:TestPoint
- R1, R2: value 4.7k -> 5.1k 1%; footprint Resistor_SMD:R_0603_1608Metric_Pad0.98x0.95mm_HandSolder -> Resistor_SMD:R_0603_1608Metric; LCSC C2907166 -> C23186
Connections:
- net +3.3V: now also C9.1, L1.2, R6.2; no longer JP4.2 (B)
- net +5V: now also C10.1, L2.2, R7.2, J9.1 (Pin_1), R28.1; no longer JP5.2 (B)
- net CC1: now also TP3.1
- net CC2: now also TP4.1
- net GND: now also U3.18 (A0), U3.23 (A1), U3.24 (A2), J9.4 (Pin_4), Q3.2 (E), R24.2, R26.2
- net PM2_TX: now also JP5.2 (B), R25.1; no longer J8.4 (Pin_4), U4.10 (MTDI/GPIO5/ADC1_CH5)
- net USB+: now also TP1.1
- net USB-: now also TP2.1
- net at J8.2 (Pin_2): now also JP5.1 (A)
- net at J8.5 (Pin_5): now also JP4.1 (A)
- net VBUS: now reaches U5.A4 (VBUS)
- net VBUS: now also U5.A9 (VBUS), U5.B4 (VBUS), U5.B9 (VBUS), TP5.1
- net PM2_RX_3.3V: now reaches U4.20 (GPIO15)
- net PM2_RX_3.3V: now also R27.1
- net IO8_EXTRA: now reaches U4.22 (GPIO8)
- net IO8_EXTRA: now also J9.2 (Pin_2)
- net IO2_EXTRA: now reaches U4.5 (GPIO2/ADC1_CH2)
- net IO2_EXTRA: now also J9.3 (Pin_3)
- net PM2_TX_3.3V: now reaches U4.6 (GPIO3/ADC1_CH3)
- net PM2_TX_3.3V: now also R25.2, R26.1
- removed net 3.3V_PRE_JUMPER: C9.1, JP4.1 (A), L1.2, R6.2
- new net: Q3.1 (B), R27.2
- new net PM2_PWM: J8.4 (Pin_4), R23.1
- new net PM2_PWM_3.3V: R23.2, R24.1, U4.10 (MTDI/GPIO5/ADC1_CH5)
- new net PM2_RX: JP4.2 (B), Q3.3 (C), R28.2
- no-connect marks 4 -> 2
Other:
- note removed: "TPS5430 - 47µH @ 550KHz"
- moved on the sheet: Q2, R20, R22
